Commit message: bug fixed

File: minibot_description/urdf/minibot.urdf.xacro (robot description, xacro)
@@ -9,5 +9,5 @@
                 <origin xyz="0 0 0" rpy="0 0 0"/>
                 <geometry>
-                    <mesh filename="file://$(find minibot_description)/meshes/visual/base_link.dae" scale="1 1 1"/>
+                    <mesh filename="package://minibot_description/meshes/visual/base_link.dae" scale="1 1 1"/>
                 </geometry>
             </visual>
@@ -15,5 +15,5 @@
                 <origin xyz="0 0 0" rpy="0 0 0"/>
                 <geometry>
-                    <mesh filename="file://$(find minibot_description)/meshes/collision/base_link.stl" scale="1 1 1"/>
+                    <mesh filename="package://minibot_description/meshes/collision/base_link.stl" scale="1 1 1"/>
                 </geometry>
             </collision>
@@ -34,5 +34,5 @@
                     <origin xyz="0 0 0" rpy="0 0 ${dir * pi/2}"/>
                     <geometry>
-                        <mesh filename="file://$(find minibot_description)/meshes/visual/wheel.dae" scale="1 1 1"/>
+                        <mesh filename="package://minibot_description/meshes/visual/wheel.dae" scale="1 1 1"/>
                     </geometry>
                 </visual>
@@ -40,5 +40,5 @@
                     <origin xyz="0 0 0" rpy="0 0 ${dir * pi/2}"/>
                     <geometry>
-                        <mesh filename="file://$(find minibot_description)/meshes/collision/wheel.stl" scale="1 1 1"/>
+                        <mesh filename="package://minibot_description/meshes/collision/wheel.stl" scale="1 1 1"/>
                     </geometry>
                 </collision>
@@ -64,5 +64,5 @@
                 <origin xyz="0 0 0" rpy="0 0 0"/>
                 <geometry>
-                    <mesh filename="file://$(find minibot_description)/meshes/visual/front_camera.dae" scale="1 1 1"/>
+                    <mesh filename="package://minibot_description/meshes/visual/front_camera.dae" scale="1 1 1"/>
                 </geometry>
             </visual>
@@ -70,5 +70,5 @@
                 <origin xyz="0 0 0" rpy="0 0 0"/>
                 <geometry>
-                    <mesh filename="file://$(find minibot_description)/meshes/collision/front_camera.stl" scale="1 1 1"/>
+                    <mesh filename="package://minibot_description/meshes/collision/front_camera.stl" scale="1 1 1"/>
                 </geometry>
             </collision>

File: minibot_description/urdf/minibot_ros2_control.urdf.xacro (robot description, xacro)
@@ -1,5 +1,5 @@
 <?xml version="1.0"?>
 <robot xmlns:xacro="http://www.ros.org/wiki/xacro">
-    <xacro:macro name="insert_ros2_control" params="prefix is_sim:=^|false">
+    <xacro:macro name="insert_ros2_control" params="prefix is_sim:=^|false port_name baudrate">
         <ros2_control name="${prefix}minibot_system" type="system">
             <xacro:if value="$(arg is_sim)">
@@ -11,6 +11,6 @@
                 <hardware>
                     <plugin>minibot_hardware/MinibotSystemHardware</plugin>
-                    <param name="port_name">/dev/ttyACM0</param>
-                    <param name="baudrate">921600</param>
+                    <param name="port_name">$(arg port_name)</param>
+                    <param name="baudrate">$(arg baudrate)</param>
                 </hardware>
             </xacro:unless>

File: minibot_description/urdf/robot.urdf.xacro (robot description, xacro)
@@ -8,9 +8,11 @@
     <xacro:arg name="is_sim" default="false"/>
     <xacro:arg name="lidar_model" default="ydlidar_x2"/> <!-- ydlidar_x2, hokuyo -->
+    <xacro:arg name="port_name" default="/dev/ttyACM0"/>
+    <xacro:arg name="baudrate" default="912600"/>
     <xacro:property name="lidar_model" value="$(arg lidar_model)"/>
     <xacro:property name="prefix" value="$(arg prefix)"/>
     <!-- insert robot base -->
     <xacro:insert_robot prefix="$(arg prefix)"/>
-    <xacro:insert_ros2_control prefix="$(arg prefix)" is_sim="$(arg is_sim)"/>
+    <xacro:insert_ros2_control prefix="$(arg prefix)" is_sim="$(arg is_sim)" port_name="$(arg port_name)" baudrate="$(arg baudrate)"/>
     <xacro:if value="$(arg is_sim)">
         <xacro:insert_gazebo prefix="$(arg prefix)" lidar_model="$(arg lidar_model)"/>
@@ -22,5 +24,5 @@
                 <origin xyz="0 0 0" rpy="0 0 0"/>
                 <geometry>
-                    <mesh filename="file://$(find minibot_description)/meshes/visual/URG-04LX-UG01.dae" scale="1 1 1"/>
+                    <mesh filename="package://minibot_description/meshes/visual/URG-04LX-UG01.dae" scale="1 1 1"/>
                 </geometry>
             </visual>
@@ -28,5 +30,5 @@
                 <origin xyz="0 0 0" rpy="0 0 0"/>
                 <geometry>
-                    <mesh filename="file://$(find minibot_description)/meshes/collision/URG-04LX-UG01.stl" scale="1 1 1"/>
+                    <mesh filename="package://minibot_description/meshes/collision/URG-04LX-UG01.stl" scale="1 1 1"/>
                 </geometry>
             </collision>

Commit message: bug fixed add simple_building.world test map building

File: minibot_description/urdf/minibot.urdf.xacro (robot description, xacro)
@@ -21,5 +21,6 @@
                 <origin xyz="0 0 0.028" rpy="0 0 0"/>
                 <mass value="2.0"/>
-                <inertia ixx="0.000213" ixy="0" ixz="0" iyy="0.007034" iyz="0" izz="0.008104"/>
+                <!-- <inertia ixx="0.000213" ixy="0" ixz="0" iyy="0.007034" iyz="0" izz="0.008104"/> -->
+                <inertia ixx="0.01" ixy="0" ixz="0" iyy="0.01" iyz="0" izz="0.01"/>
             </inertial>
         </link>
@@ -55,5 +56,5 @@
                 <child link="${prefix}${prefix_dir}_wheel"/>
                 <axis xyz="0 1 0"/>
-                <origin xyz="0 ${dir * wheel_speration/2} 0" rpy="0 0 0"/>
+                <origin xyz="0 ${dir * wheel_speration/2} -0.0001" rpy="0 0 0"/>
             </joint>
         </xacro:macro>

File: minibot_description/urdf/minibot_gazebo.urdf.xacro (robot description, xacro)
@@ -22,6 +22,6 @@
         </gazebo>
         <gazebo reference="${prefix}base_link">
-            <mu1>0.01</mu1>
-            <mu2>0.01</mu2>
+            <mu1>0.0</mu1>
+            <mu2>0.0</mu2>
             <!-- <minDepth>0.001</minDepth> -->
         </gazebo>

Commit message: Change the robot model

File: minibot_description/urdf/minibot.urdf.xacro (robot description, xacro)
@@ -3,5 +3,5 @@
     <xacro:macro name="insert_robot" params="prefix">
         <xacro:property name="wheel_diameter" value="0.068"/>
-        <xacro:property name="wheel_speration" value="0.1736"/>
+        <xacro:property name="wheel_speration" value="0.180"/>
         <link name="${prefix}base_footprint"/>
         <link name="${prefix}base_link">
@@ -19,5 +19,5 @@
             </collision>
             <inertial>
-                <origin xyz="0 0 0.028" rpy="0 0 0"/>
+                <origin xyz="-0.02 0 0.028" rpy="0 0 0"/>
                 <mass value="2.0"/>
                 <!-- <inertia ixx="0.000213" ixy="0" ixz="0" iyy="0.007034" iyz="0" izz="0.008104"/> -->
@@ -56,5 +56,5 @@
                 <child link="${prefix}${prefix_dir}_wheel"/>
                 <axis xyz="0 1 0"/>
-                <origin xyz="0 ${dir * wheel_speration/2} -0.0001" rpy="0 0 0"/>
+                <origin xyz="0 ${dir * wheel_speration/2} 0" rpy="0 0 0"/>
             </joint>
         </xacro:macro>
@@ -83,5 +83,5 @@
             <parent link="${prefix}base_link"/>
             <child link="${prefix}front_camera_mount"/>
-            <origin xyz="0.0864 0 0.0355" rpy="0 0 0"/>
+            <origin xyz="0.045 0 0.085" rpy="0 0 0"/>
         </joint>
         <link name="${prefix}camera_link"/>
@@ -91,4 +91,34 @@
             <origin xyz="0.0111 0 0.0193" rpy="0 ${pi/2} 0"/>
         </joint>
+        <link name="${prefix}ul_sensor_mount">
+            <visual>
+                <origin xyz="0 0 0" rpy="0 0 0"/>
+                <geometry>
+                    <mesh filename="package://minibot_description/meshes/visual/ul_sensor.dae" scale="1 1 1"/>
+                </geometry>
+            </visual>
+            <collision>
+                <origin xyz="0 0 0" rpy="0 0 0"/>
+                <geometry>
+                    <mesh filename="package://minibot_description/meshes/collision/ul_sensor.stl" scale="1 1 1"/>
+                </geometry>
+            </collision>
+            <inertial>
+                <origin xyz="0.005 0 0.013" rpy="0 0 0"/>
+                <mass value="0.050000"/>
+                <inertia ixx="0.000005" ixy="0" ixz="-0.000001" iyy="0.000004" iyz="0" izz="0.000003"/>
+            </inertial>
+        </link>
+        <joint name="${prefix}ul_sensor_mount_fixed_joint" type="fixed">
+            <parent link="${prefix}base_link"/>
+            <child link="${prefix}ul_sensor_mount"/>
+            <origin xyz="0.03 0 0.01" rpy="0 0 0"/>
+        </joint>
+        <link name="${prefix}ul_sensor_link"/>
+        <joint name="${prefix}ul_sensor_link_fixed_joint" type="fixed">
+            <parent link="${prefix}ul_sensor_mount"/>
+            <child link="${prefix}ul_sensor_link"/>
+            <origin xyz="0.02 0 0" rpy="0 0 0"/>
+        </joint>
     </xacro:macro>
 </robot>

File: minibot_description/urdf/minibot_gazebo.urdf.xacro (robot description, xacro)
@@ -1,5 +1,5 @@
 <?xml version="1.0"?>
 <robot xmlns:xacro="http://www.ros.org/wiki/xacro">
-    <xacro:macro name="insert_gazebo" params="prefix lidar_model">
+    <xacro:macro name="insert_gazebo" params="prefix">
         <gazebo>
             <plugin filename="libgazebo_ros2_control.so" name="gazebo_ros2_control">
@@ -27,40 +27,23 @@
         </gazebo>
         <gazebo reference="${prefix}laser_link">
-            <sensor name="laser" type="ray">
+            <sensor name="laser" type="gpu_ray">
                 <pose>0 0 0 0 0 0</pose>
                 <always_on>1</always_on>
                 <update_rate>15</update_rate>
-                <visualize>true</visualize>
+                <visualize>false</visualize>
                 <ray>
-                    <xacro:if value="${lidar_model == 'hokuyo'}">
-                        <scan>
-                            <horizontal>
-                                <samples>666</samples>
-                                <resolution>1</resolution>
-                                <min_angle>${-120*pi/180}</min_angle>
-                                <max_angle>${120*pi/180}</max_angle>
-                            </horizontal>
-                        </scan>
-                        <range>
-                            <min>0.02</min>
-                            <max>5.0</max>
-                            <resolution>0.03</resolution>
-                        </range>
-                    </xacro:if>
-                    <xacro:if value="${lidar_model == 'ydlidar_x2'}">
-                        <scan>
-                            <horizontal>
-                                <samples>375</samples>
-                                <resolution>1</resolution>
-                                <min_angle>${-180*pi/180}</min_angle>
-                                <max_angle>${180*pi/180}</max_angle>
-                            </horizontal>
-                        </scan>
-                        <range>
-                            <min>0.12</min>
-                            <max>8.0</max>
-                            <resolution>0.05</resolution>
-                        </range>
-                    </xacro:if>
+                    <scan>
+                        <horizontal>
+                            <samples>375</samples>
+                            <resolution>1</resolution>
+                            <min_angle>${-180*pi/180}</min_angle>
+                            <max_angle>${180*pi/180}</max_angle>
+                        </horizontal>
+                    </scan>
+                    <range>
+                        <min>0.12</min>
+                        <max>8.0</max>
+                        <resolution>0.05</resolution>
+                    </range>
                     <noise>
                         <type>gaussian</type>

File: minibot_description/urdf/minibot_ros2_control.urdf.xacro (robot description, xacro)
@@ -1,5 +1,5 @@
 <?xml version="1.0"?>
 <robot xmlns:xacro="http://www.ros.org/wiki/xacro">
-    <xacro:macro name="insert_ros2_control" params="prefix is_sim:=^|false port_name baudrate">
+    <xacro:macro name="insert_ros2_control" params="prefix is_sim:=^|false robot_port_name robot_baudrate">
         <ros2_control name="${prefix}minibot_system" type="system">
             <xacro:if value="$(arg is_sim)">
@@ -11,6 +11,6 @@
                 <hardware>
                     <plugin>minibot_hardware/MinibotSystemHardware</plugin>
-                    <param name="port_name">$(arg port_name)</param>
-                    <param name="baudrate">$(arg baudrate)</param>
+                    <param name="port_name">$(arg robot_port_name)</param>
+                    <param name="baudrate">$(arg robot_baudrate)</param>
                 </hardware>
             </xacro:unless>

File: minibot_description/urdf/robot.urdf.xacro (robot description, xacro)
@@ -7,80 +7,44 @@
     <xacro:arg name="prefix" default=""/>
     <xacro:arg name="is_sim" default="false"/>
-    <xacro:arg name="lidar_model" default="ydlidar_x2"/> <!-- ydlidar_x2, hokuyo -->
-    <xacro:arg name="port_name" default="/dev/ttyACM0"/>
-    <xacro:arg name="baudrate" default="912600"/>
-    <xacro:property name="lidar_model" value="$(arg lidar_model)"/>
+    <xacro:arg name="robot_port_name" default="/dev/ttyArduino"/>
+    <xacro:arg name="robot_baudrate" default="500000"/>
     <xacro:property name="prefix" value="$(arg prefix)"/>
     <!-- insert robot base -->
     <xacro:insert_robot prefix="$(arg prefix)"/>
-    <xacro:insert_ros2_control prefix="$(arg prefix)" is_sim="$(arg is_sim)" port_name="$(arg port_name)" baudrate="$(arg baudrate)"/>
+    <xacro:insert_ros2_control prefix="$(arg prefix)" is_sim="$(arg is_sim)" robot_port_name="$(arg robot_port_name)" robot_baudrate="$(arg robot_baudrate)"/>
     <xacro:if value="$(arg is_sim)">
-        <xacro:insert_gazebo prefix="$(arg prefix)" lidar_model="$(arg lidar_model)"/>
-    </xacro:if>
-    <!-- insert hokuyo lidar -->
-    <xacro:if value="${lidar_model == 'hokuyo'}">
-        <link name="${prefix}hokuyo_lidar_mount">
-            <visual>
-                <origin xyz="0 0 0" rpy="0 0 0"/>
-                <geometry>
-                    <mesh filename="package://minibot_description/meshes/visual/URG-04LX-UG01.dae" scale="1 1 1"/>
-                </geometry>
-            </visual>
-            <collision>
-                <origin xyz="0 0 0" rpy="0 0 0"/>
-                <geometry>
-                    <mesh filename="package://minibot_description/meshes/collision/URG-04LX-UG01.stl" scale="1 1 1"/>
-                </geometry>
-            </collision>
-            <inertial>
-                <origin xyz="0 0 0.031" rpy="0 0 0"/>
-                <mass value="0.200"/>
-                <inertia ixx="0.0001089" ixy="0" ixz="0.000001" iyy="0.0001094" iyz="0" izz="0.0000720"/>
-            </inertial>
-        </link>
-        <joint name="${prefix}hokuyo_lidar_mount_fixed_joint" type="fixed">
-            <parent link="${prefix}base_link"/>
-            <child link="${prefix}hokuyo_lidar_mount"/>
-            <origin xyz="0.02 0 0.08705" rpy="0 0 0"/>
-        </joint>
-        <link name="${prefix}laser_link"/>
-        <joint name="${prefix}laser_link_fixed_joint" type="fixed">
-            <parent link="${prefix}hokuyo_lidar_mount"/>
-            <child link="${prefix}laser_link"/>
-            <origin xyz="0 0 0.06" rpy="0 0 0"/>
-        </joint>
+        <xacro:insert_gazebo prefix="$(arg prefix)"/>
     </xacro:if>
     <!-- insert ydlidar_x2 lidar -->
-    <xacro:if value="${lidar_model == 'ydlidar_x2'}">
-        <link name="${prefix}ydlidar_lidar_mount">
-            <visual>
-                <origin xyz="0 0 0" rpy="0 0 0"/>
-                <geometry>
-                    <mesh filename="file://$(find minibot_description)/meshes/visual/ydlidar_x2_assy.dae" scale="1 1 1"/>
-                </geometry>
-            </visual>
-            <collision>
-                <origin xyz="0 0 0" rpy="0 0 0"/>
-                <geometry>
-                    <mesh filename="file://$(find minibot_description)/meshes/collision/ydlidar_x2_assy.stl" scale="1 1 1"/>
-                </geometry>
-            </collision>
-            <inertial>
-                <origin xyz="0.007 0 0.025" rpy="0 0 0"/>
-                <mass value="0.150"/>
-                <inertia ixx="0.000058" ixy="0" ixz="0.000005" iyy="0.000099" iyz="0" izz="0.000103"/>
-            </inertial>
-        </link>
-        <joint name="${prefix}hokuyo_lidar_mount_fixed_joint" type="fixed">
-            <parent link="${prefix}base_link"/>
-            <child link="${prefix}ydlidar_lidar_mount"/>
-            <origin xyz="0 0 0.08705" rpy="0 0 0"/>
-        </joint>
-        <link name="${prefix}laser_link"/>
-        <joint name="${prefix}laser_link_fixed_joint" type="fixed">
-            <parent link="${prefix}ydlidar_lidar_mount"/>
-            <child link="${prefix}laser_link"/>
-            <origin xyz="0 0 0.04245" rpy="0 0 0"/>
-        </joint>
-    </xacro:if>
+    <link name="${prefix}ydlidar_lidar_mount">
+        <visual>
+            <origin xyz="0 0 0" rpy="0 0 0"/>
+            <geometry>
+                <mesh filename="file://$(find minibot_description)/meshes/visual/ydlidar_x2_assy.dae" scale="1 1 1"/>
+            </geometry>
+        </visual>
+        <collision>
+            <origin xyz="0 0 0" rpy="0 0 0"/>
+            <geometry>
+                <mesh filename="file://$(find minibot_description)/meshes/collision/ydlidar_x2_assy.stl" scale="1 1 1"/>
+            </geometry>
+        </collision>
+        <inertial>
+            <origin xyz="0.007 0 0.025" rpy="0 0 0"/>
+            <mass value="0.150"/>
+            <!-- <inertia ixx="0.000058" ixy="0" ixz="0.000005" iyy="0.000099" iyz="0" izz="0.000103"/> -->
+            <inertia ixx="0.0058" ixy="0" ixz="0.0005" iyy="0.0099" iyz="0" izz="0.0103"/>
+        </inertial>
+    </link>
+    <joint name="${prefix}idar_mount_fixed_joint" type="fixed">
+        <parent link="${prefix}base_link"/>
+        <child link="${prefix}ydlidar_lidar_mount"/>
+        <origin xyz="-0.01 0 0.085" rpy="0 0 0"/>
+    </joint>
+    <link name="${prefix}laser_link"/>
+    <joint name="${prefix}laser_link_fixed_joint" type="fixed">
+        <parent link="${prefix}ydlidar_lidar_mount"/>
+        <child link="${prefix}laser_link"/>
+        <origin xyz="0 0 0.04245" rpy="0 0 0"/>
+    </joint>
 </robot>
