Commit message: bug fixed

File: minibot_description/urdf/robot.urdf.xacro (robot description, xacro)
@@ -21,5 +21,5 @@
             <origin xyz="0 0 0" rpy="0 0 0"/>
             <geometry>
-                <mesh filename="file://$(find minibot_description)/meshes/visual/ydlidar_x2_assy.dae" scale="1 1 1"/>
+                <mesh filename="package://minibot_description/meshes/visual/ydlidar_x2_assy.dae" scale="1 1 1"/>
             </geometry>
         </visual>
@@ -27,5 +27,5 @@
             <origin xyz="0 0 0" rpy="0 0 0"/>
             <geometry>
-                <mesh filename="file://$(find minibot_description)/meshes/collision/ydlidar_x2_assy.stl" scale="1 1 1"/>
+                <mesh filename="package://minibot_description/meshes/collision/ydlidar_x2_assy.stl" scale="1 1 1"/>
             </geometry>
         </collision>

Commit message: param changed

File: minibot_description/urdf/robot.urdf.xacro (robot description, xacro)
@@ -33,6 +33,5 @@
             <origin xyz="0.007 0 0.025" rpy="0 0 0"/>
             <mass value="0.150"/>
-            <!-- <inertia ixx="0.000058" ixy="0" ixz="0.000005" iyy="0.000099" iyz="0" izz="0.000103"/> -->
-            <inertia ixx="0.0058" ixy="0" ixz="0.0005" iyy="0.0099" iyz="0" izz="0.0103"/>
+            <inertia ixx="0.000058" ixy="0" ixz="0.000005" iyy="0.000099" iyz="0" izz="0.000103"/>
         </inertial>
     </link>
